Commit message: Add files via upload

File: mobile_manipulator_body/mobile_manipulator_body/urdf/robot_base.urdf (robot description, URDF)
Before this commit: robot mobile_manipulator, 6 links, 5 joints
Links:
- added link camera_frame; visual box size=0.04 0.04 0.04
Joints:
- added joint camera_joint: type fixed, parent base_link, child camera_frame, origin xyz=0.34 0 0.05 rpy=0 0 0
